File: memory/8-bit-memory-tht/8-bit-memory-tht.sch (KiCad schematic (older format))
At the start: 126 parts, among them J1 J1-1_bit_bus, J2 J8-8_bit_bus_connector, J3 J2-2_pole_connector, J4 J8-8_bit_bus_connector, Q1 2N7000, Q10 2N7000, Q11 2N7000, Q12 2N7000, Q13 2N7000, Q14 2N7000, Q15 2N7000, Q16 2N7000, Q17 2N7000, Q18 2N7000, Q19 2N7000, Q2 2N7000, Q20 2N7000, Q21 2N7000, Q22 2N7000, Q23 2N7000, Q24 2N7000, Q25 2N7000, Q26 2N7000, Q27 2N7000, Q28 2N7000, Q29 2N7000, Q3 2N7000, Q30 2N7000, Q31 2N7000, Q32 2N7000, Q33 2N7000, Q34 2N7000, Q35 2N7000, Q36 2N7000, Q37 2N7000, Q38 2N7000, Q39 2N7000, Q4 2N7000, Q40 2N7000, Q41 2N7000, Q42 2N7000, Q43 2N7000, Q44 2N7000, Q45 2N7000, Q46 2N7000, Q47 2N7000, Q48 2N7000, Q49 2N7000, Q5 2N7000, Q50 2N7000, Q51 2N7000, Q52 2N7000, Q53 2N7000, Q54 2N7000, Q55 2N7000, Q56 2N7000, Q57 2N7000, Q58 2N7000, Q59 2N7000, Q6 2N7000, Q60 2N7000, Q61 2N7000, Q62 2N7000, Q63 2N7000, Q64 2N7000, Q65 2N7000, Q66 2N7000, Q67 2N7000, Q68 2N7000, Q69 2N7000, Q7 2N7000, Q70 2N7000, Q71 2N7000, Q72 2N7000, Q73 2N7000, Q8 2N7000, Q9 2N7000

Commit message: Finish THT memory board layout
Parts:
- J1: footprint emlun:J1-1_bit_bus -> emlun:J1x2-double_1_bit_bus
- J2, J4: footprint emlun:J8-8_bit_bus_connector -> emlun:J8x2-double_8_bit_bus_connector
- J3: footprint emlun:J2-2_pole_connector -> emlun:J2x2-double_2_pole_connector
- Q1, Q10, Q11, Q12, Q13, Q14, Q15, Q16, Q17, Q18, Q19, Q2, Q20, Q21, Q22, Q23, Q24, Q25, Q26, Q27, Q28, Q29, Q3, Q30, Q31, Q32, Q33, Q34, Q35, Q36, Q37, Q38, Q39, Q4, Q40, Q41, Q42, Q43, Q44, Q45, Q46, Q47, Q48, Q49, Q5, Q50, Q51, Q52, Q53, Q54, Q55, Q56, Q57, Q58, Q59, Q6, Q60, Q61, Q62, Q63, Q64, Q65, Q66, Q67, Q68, Q69, Q7, Q70, Q71, Q72, Q73, Q8, Q9: footprint TO_SOT_Packages_SMD:SOT-23 -> electrokit:TO-92_Molded_Wide_Inline
- R1, R10, R11, R12, R13, R14, R15, R16, R17, R18, R19, R2, R20, R21, R22, R23, R24, R25, R26, R27, R28, R29, R3, R30, R31, R32, R33, R34, R35, R36, R37, R38, R39, R4, R40, R41, R42, R43, R44, R45, R46, R47, R48, R49, R5, R6, R7, R8, R9: footprint Resistors_SMD:R_0805 -> emlun:R_Axial_DIN0204_L3.6mm_D1.6mm_P5.08mm_Horizontal
