File: memory/8-bit-memory-tht/8-bit-memory-tht.sch (KiCad schematic (older format))
At the start: 211 parts, among them J1 J1-1_bit_bus, J2 J8-8_bit_bus_connector, J3 J8-8_bit_bus_connector, J4 PWR-2_pole_power_connector, Q1 2N7000, Q10 2N7000, Q100 2N7000, Q101 2N7000, Q102 2N7000, Q103 2N7000, Q104 2N7000, Q105 2N7000, Q106 2N7000, Q11 2N7000, Q12 2N7000, Q13 2N7000, Q14 2N7000, Q15 2N7000, Q16 2N7000, Q17 2N7000, Q18 2N7000, Q19 2N7000, Q2 2N7000, Q20 2N7000, Q21 2N7000, Q22 2N7000, Q23 2N7000, Q24 2N7000, Q25 2N7000, Q26 2N7000, Q27 2N7000, Q28 2N7000, Q29 2N7000, Q3 2N7000, Q30 2N7000, Q31 2N7000, Q32 2N7000, Q33 2N7000, Q34 2N7000, Q35 2N7000, Q36 2N7000, Q37 2N7000, Q38 2N7000, Q39 2N7000, Q4 2N7000, Q40 2N7000, Q41 2N7000, Q42 2N7000, Q43 2N7000, Q44 2N7000, Q45 2N7000, Q46 2N7000, Q47 2N7000, Q48 2N7000, Q49 2N7000, Q5 2N7000, Q50 2N7000, Q51 2N7000, Q52 2N7000, Q53 2N7000, Q54 2N7000, Q55 2N7000, Q56 2N7000, Q57 2N7000, Q58 2N7000, Q59 2N7000, Q6 2N7000, Q60 2N7000, Q61 2N7000, Q62 2N7000, Q63 2N7000, Q64 2N7000, Q65 2N7000, Q66 2N7000, Q67 2N7000, Q68 2N7000, Q69 2N7000, Q7 2N7000, Q70 2N7000, Q71 2N7000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

Commit message: Rescue old components
Parts:
- J1: symbol emlun:J1-1_bit_bus -> 8-bit-memory-tht-rescue:J1-1_bit_bus-emlun
- J2, J3: symbol emlun:J8-8_bit_bus_connector -> 8-bit-memory-tht-rescue:J8-8_bit_bus_connector-emlun
- J4: symbol emlun:PWR-2_pole_power_connector -> 8-bit-memory-tht-rescue:PWR-2_pole_power_connector-emlun
Changed lines of the file:
@@
 I0
 $Comp
-L emlun:J8-8_bit_bus_connector J2
+L 8-bit-memory-tht-rescue:J8-8_bit_bus_connector-emlun J2
 U 1 1 59C7FAF8
 P 1500 2150
@@
 $EndComp
 $Comp
-L emlun:J1-1_bit_bus J1
+L 8-bit-memory-tht-rescue:J1-1_bit_bus-emlun J1
 U 1 1 59C7FD55
 P 1500 1600
@@
 	6200 3450 6200 2500
 $Comp
-L emlun:J8-8_bit_bus_connector J3
+L 8-bit-memory-tht-rescue:J8-8_bit_bus_connector-emlun J3
 U 1 1 59C81A4F
 P 8250 2150
@@
 $EndComp
 $Comp
-L emlun:PWR-2_pole_power_connector J4
+L 8-bit-memory-tht-rescue:PWR-2_pole_power_connector-emlun J4
 U 1 1 5B3A72AC
 P 1500 2750
@@
 Wire Wire Line
 	9700 19650 9700 21200
+Connection ~ 8100 19650
 Wire Bus Line
 	2000 1800 2000 15650
-Connection ~ 8100 19650
 $EndSCHEMATC
