File: 8-bit-adder/8-bit-adder.sch (KiCad schematic (older format))
At the start: 223 parts, among them J1 J2-2_pole_connector, J2 J1-1_bit_bus, J3 J8-8_bit_bus_connector, J4 J8-8_bit_bus_connector, J5 J1-1_bit_bus, J6 J8-8_bit_bus_connector, Q1 2N7000, Q10 2N7000, Q100 2N7000, Q101 2N7000, Q102 2N7000, Q103 2N7000, Q104 2N7000, Q105 2N7000, Q106 2N7000, Q107 2N7000, Q108 2N7000, Q109 2N7000, Q11 2N7000, Q110 2N7000, Q111 2N7000, Q112 2N7000, Q113 2N7000, Q114 2N7000, Q115 2N7000, Q116 2N7000, Q117 2N7000, Q118 2N7000, Q119 2N7000, Q12 2N7000, Q120 2N7000, Q121 2N7000, Q122 2N7000, Q123 2N7000, Q124 2N7000, Q125 2N7000, Q126 2N7000, Q127 2N7000, Q128 2N7000, Q13 2N7000, Q14 2N7000, Q15 2N7000, Q16 2N7000, Q17 2N7000, Q18 2N7000, Q19 2N7000, Q2 2N7000, Q20 2N7000, Q21 2N7000, Q22 2N7000, Q23 2N7000, Q24 2N7000, Q25 2N7000, Q26 2N7000, Q27 2N7000, Q28 2N7000, Q29 2N7000, Q3 2N7000, Q30 2N7000, Q31 2N7000, Q32 2N7000, Q33 2N7000, Q34 2N7000, Q35 2N7000, Q36 2N7000, Q37 2N7000, Q38 2N7000, Q39 2N7000, Q4 2N7000, Q40 2N7000, Q41 2N7000, Q42 2N7000, Q43 2N7000, Q44 2N7000, Q45 2N7000, Q46 2N7000, Q47 2N7000, Q48 2N7000, Q49 2N7000, Q5 2N7000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

Commit message: Update adder circuit to revision 2
Parts:
- removed J1: J2-2_pole_connector, emlun:J2-2_pole_connector, symbol J2-2_pole_connector
- removed J5: J1-1_bit_bus, emlun:J1-1_bit_bus, symbol J1-1_bit_bus
- added J1: PWR-2_pole_power_connector, emlun:J2x2-double_2_pole_connector, symbol PWR-2_pole_power_connector
- added J5: J2-2_bit_bus, emlun:J2x2-double_2_bit_bus, symbol J2-2_bit_bus
- added Q129, Q130, Q131, Q132, Q133, Q134, Q135: 2N7000, electrokit:TO-92_Molded_Wide_Inline, symbol 2N7000
- added R90, R91, R92, R93: 1M, emlun:R_Axial_DIN0204_L3.6mm_D1.6mm_P5.08mm_Horizontal, symbol R
- J2: footprint emlun:J1-1_bit_bus -> emlun:J1x2-double_1_bit_bus
- J3, J4, J6: footprint emlun:J8-8_bit_bus_connector -> emlun:J8x2-double_8_bit_bus_connector
- R1, R10, R11, R12, R13, R14, R15, R16, R17, R18, R19, R2, R20, R21, R22, R23, R24, R25, R26, R27, R28, R29, R3, R30, R31, R32, R33, R34, R35, R36, R37, R38, R39, R4, R40, R41, R42, R43, R44, R45, R46, R47, R48, R49, R5, R50, R51, R52, R53, R54, R55, R56, R57, R58, R59, R6, R60, R61, R62, R63, R64, R65, R66, R67, R68, R69, R7, R70, R71, R72, R73, R74, R75, R76, R77, R78, R79, R8, R80, R81, R82, R83, R84, R85, R86, R87, R88, R89, R9: footprint Resistors_THT:R_Axial_DIN0204_L3.6mm_D1.6mm_P5.08mm_Horizontal -> emlun:R_Axial_DIN0204_L3.6mm_D1.6mm_P5.08mm_Horizontal
Connections:
- net C6: now also Q129.2 (G), Q133.2 (G)
- net C7: now also J5.1, Q130.2 (G), Q134.2 (G)
- net GND: now also J1.1 (GND), Q129.1 (S), Q130.1 (S), Q131.1 (S), Q132.1 (S), Q133.1 (S), Q135.1 (S)
- net VCC: now also J1.2 (VCC), R90.1, R91.1, R92.1, R93.1
- new net: Q129.3 (D), Q130.3 (D), Q131.2 (G), R90.2
- new net: Q133.3 (D), Q134.1 (S)
- new net: Q134.3 (D), Q135.2 (G), R92.2
- new net: Q132.2 (G), Q135.3 (D), R93.2
- new net Os: J5.2, Q131.3 (D), Q132.3 (D), R91.2
