File: bus-selector/bus-selector.kicad_pcb (KiCad board)
At the start: 2 copper layers, 219 parts, among them J1 Conn_01x08, J2 Conn_01x08, J3 Conn_01x08, J4 Conn_01x08, J5 Conn_01x02, J6 Conn_01x08, J7 PWR-2_pole_power_connector, Q1 2N7000, Q10 2N7000, Q11 2N7000, Q12 2N7000, Q13 2N7000, Q14 2N7000, Q15 2N7000, Q16 2N7000, Q17 2N7000, Q18 2N7000, Q19 2N7000, Q2 2N7000, Q20 2N7000, Q21 2N7000, Q22 2N7000, Q23 2N7000, Q24 2N7000, Q25 2N7000, Q26 2N7000, Q27 2N7000, Q28 2N7000, Q29 2N7000, Q3 2N7000, Q30 2N7000, Q31 2N7000, Q32 2N7000, Q33 2N7000, Q34 2N7000, Q35 2N7000, Q36 2N7000, Q37 2N7000, Q38 2N7000, Q39 2N7000, Q4 2N7000, Q40 2N7000, Q41 2N7000, Q42 2N7000, Q43 2N7000, Q44 2N7000, Q45 2N7000, Q46 2N7000, Q47 2N7000, Q48 2N7000, Q49 2N7000, Q5 2N7000, Q50 2N7000, Q51 2N7000, Q52 2N7000, Q53 2N7000, Q54 2N7000, Q55 2N7000, Q56 2N7000, Q57 2N7000, Q58 2N7000, Q59 2N7000, Q6 2N7000, Q60 2N7000, Q61 2N7000, Q62 2N7000, Q63 2N7000, Q64 2N7000, Q65 2N7000, Q66 2N7000, Q67 2N7000, Q68 2N7000, Q69 2N7000, Q7 2N7000, Q70 2N7000, Q71 2N7000, Q72 2N7000, Q73 2N7000, Q74 2N7000, Q75 2N7000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

Commit message: Finish PCB layout of bus selector
Parts:
- added REF**: MountingHole_2.2mm_M2_Pad, MountingHole:MountingHole_2.2mm_M2_Pad, F.Cu at (146.1, 19.1)
- added REF**: MountingHole_2.2mm_M2_Pad, MountingHole:MountingHole_2.2mm_M2_Pad, F.Cu at (21.6, 19.1)
- added REF**: MountingHole_2.2mm_M2_Pad, MountingHole:MountingHole_2.2mm_M2_Pad, F.Cu at (146.1, 77.5)
- added REF**: MountingHole_2.2mm_M2_Pad, MountingHole:MountingHole_2.2mm_M2_Pad, F.Cu at (21.6, 77.5)
- moved Q55 82.9 mm to (33.0, 61.0)
- moved R23 82.1 mm to (38.1, 63.5)
- moved R10 77.6 mm to (115.6, 78.7)
- moved R8 77.6 mm to (115.6, 71.1)
- moved Q50 70.6 mm to (43.2, 61.0)
- moved R21 70.6 mm to (47.0, 63.5)
- moved Q45 57.1 mm to (55.9, 61.0)
- moved R19 56.4 mm to (61.0, 63.5)
- moved R12 55.5 mm to (92.7, 71.1)
- moved R14 55.5 mm to (92.7, 78.7)
- moved Q47 52.4 mm to (50.8, 68.6)
- moved Q52 52.4 mm to (50.8, 76.2)
- moved Q49 50.6 mm to (96.5, 68.6)
- moved Q54 50.6 mm to (96.5, 76.2)
- moved Q48 48.3 mm to (73.7, 68.6)
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Routing:
- net VCC: track 7.85 -> 333.8 mm
- net GND: track 266.0 -> 409.3 mm, vias 2 -> 10
- net Net-(Q46-Pad3): track 0.00 -> 103.6 mm, vias 0 -> 5
- net /o7: track 36.5 -> 129.7 mm
- net Net-(Q51-Pad3): track 0.00 -> 91.9 mm, vias 0 -> 5
- net Net-(Q21-Pad3): track 0.00 -> 90.1 mm, vias 0 -> 4
- net Net-(Q31-Pad3): track 0.00 -> 89.4 mm, vias 0 -> 1
- net Net-(Q41-Pad3): track 0.00 -> 86.4 mm
- net /o6: track 36.5 -> 122.4 mm, vias 1 -> 2
- net Net-(Q26-Pad3): track 0.00 -> 85.6 mm, vias 0 -> 3
- net Net-(Q16-Pad3): track 0.00 -> 85.0 mm, vias 0 -> 1
- net Net-(Q36-Pad3): track 0.00 -> 76.5 mm
- net /o5: track 36.5 -> 112.6 mm, vias 1 -> 2
- net /o4: track 36.5 -> 105.4 mm, vias 1 -> 2
- net /o3: track 36.5 -> 95.6 mm, vias 1 -> 2
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- removed copper zone on B.Cu, net GND
- removed copper zone on F.Cu, net VCC
Other:
- board outline added: 129.5 x 63.5 mm
- board text added: "4-way 8 bit bus selector v1 O = s(S) s(00) = A s(01) = B s(10) = C s(11) = D Emil Lundberg emil@emlun.se 2018-07-18"
- board text added: "Production: https://PCBS.io"
