File: bus-selector/bus-selector.sch (KiCad schematic (older format))
At the start: 50 parts, among them J1 Conn_01x08, J2 Conn_01x08, J3 Conn_01x08, J4 Conn_01x08, J5 Conn_01x04, J6 Conn_01x08, J7 PWR-2_pole_power_connector, U1 74LVC1G27, U10 74AHC1G00, U11 74AHC1G00, U12 74AHC1G00, U13 74AHC1G00, U14 74AHC1G00, U15 74AHC1G00, U16 74AHC1G00, U17 74AHC1G00, U18 74AHC1G00, U19 74AHC1G00, U2 74LVC1G27, U20 74AHC1G00, U21 74AHC1G00, U22 74AHC1G00, U23 74AHC1G00, U24 74AHC1G00, U25 74AHC1G00, U26 74AHC1G00, U27 74AHC1G00, U28 74AHC1G00, U29 74AHC1G00, U3 74LVC1G27, U30 74AHC1G00, U31 74AHC1G00, U32 74AHC1G00, U33 74AHC1G00, U34 74AHC1G00, U35 74AHC1G00, U36 74AHC1G00, U37 74AHC1G00, U38 74AHC1G00, U39 74AHC1G00, U4 4002, U40 4002, U41 4002, U42 4002, U43 4002, U5 74AHC1G08, U6 74AHC1G08, U7 74LVC1G11, U8 74AHC1G00, U9 74AHC1G00

Commit message: Finish bus selector connection diagram
Parts:
- removed J5: Conn_01x04, symbol Connector_Generic:Conn_01x04
- removed U1, U2, U3: 74LVC1G27, symbol 74xGxx:74LVC1G27
- removed U10, U11, U12, U13, U14, U15, U16, U17, U18, U19, U20, U21, U22, U23, U24, U25, U26, U27, U28, U29, U30, U31, U32, U33, U34, U35, U36, U37, U38, U39, U8, U9: 74AHC1G00, symbol 74xGxx:74AHC1G00
- removed U4, U40, U41, U42, U43: 4002, symbol 4xxx:4002
- removed U5, U6: 74AHC1G08, symbol 74xGxx:74AHC1G08
- removed U7: 74LVC1G11, symbol 74xGxx:74LVC1G11
- added D1, D10, D11, D12, D13, D14, D15, D16, D17, D18, D19, D2, D20, D21, D22, D23, D24, D25, D26, D27, D28, D29, D3, D30, D31, D32, D33, D34, D35, D36, D37, D38, D39, D4, D40, D41, D42, D43, D44, D5, D6, D7, D8, D9: LED, LED_SMD:LED_0805_2012Metric_Castellated, symbol Device:LED
- added J5: Conn_01x02, emlun:J2x2-double_2_bit_bus, symbol Connector_Generic:Conn_01x02
- added Q1, Q10, Q11, Q12, Q13, Q14, Q15, Q16, Q17, Q18, Q19, Q2, Q20, Q21, Q22, Q23, Q24, Q25, Q26, Q27, Q28, Q29, Q3, Q30, Q31, Q32, Q33, Q34, Q35, Q36, Q37, Q38, Q39, Q4, Q40, Q41, Q42, Q43, Q44, Q45, Q46, Q47, Q48, Q49, Q5, Q50, Q51, Q52, Q53, Q54, Q55, Q56, Q57, Q58, Q59, Q6, Q60, Q61, Q62, Q63, Q64, Q65, Q66, Q67, Q68, Q69, Q7, Q70, Q71, Q72, Q73, Q74, Q75, Q76, Q77, Q78, Q79, Q8, Q80, Q81, Q82, Q83, Q9: 2N7000, electrokit:TO-92_Molded_Wide_Inline, symbol Transistor_FET:2N7000
- added Q100, Q101, Q102, Q103, Q104, Q105, Q106, Q107, Q108, Q109, Q110, Q111, Q112, Q113, Q114, Q115, Q116, Q117, Q118, Q119, Q120, Q121, Q122, Q123, Q124, Q125, Q126, Q127, Q84, Q85, Q86, Q87, Q88, Q89, Q90, Q91, Q92, Q93, Q94, Q95, Q96, Q97, Q98, Q99: 2N7000, Package_TO_SOT_SMD:SOT-23_Handsoldering, symbol Transistor_FET:2N7000
- added R1, R10, R11, R12, R13, R14, R15, R16, R17, R18, R19, R2, R20, R21, R22, R23, R3, R4, R5, R6, R7, R8, R9: R, emlun:R_Axial_DIN0204_L3.6mm_D1.6mm_P5.08mm_Horizontal, symbol Device:R
- added R24, R25, R26, R27, R28, R29, R30, R31, R32, R33, R34, R35, R36, R37, R38, R39, R40, R41, R42, R43, R44, R45, R46, R47, R48, R49, R50, R51, R52, R53, R54, R55, R56, R57, R58, R59, R60, R61, R62, R63, R64, R65, R66, R67: R, Resistor_SMD:R_0805_2012Metric_Pad1.29x1.40mm_HandSolder, symbol Device:R
- J1, J2, J3, J4, J6: footprint (none) -> emlun:J8x2-double_8_bit_bus_connector_1_indexed
- J7: footprint (none) -> emlun:J2x2-double_2_pole_connector
Connections:
- net labels added: sa, sb, sc, sd
- net labels removed: act_a, act_b, act_c, act_d, ao0, ao1, ao2, ao3, ao4, ao5, ao6, ao7, bo0, bo1, bo2, bo3, bo4, bo5, bo6, bo7, co0, co1, co2, co3, co4, co5, co6, co7, do0, do1, do2, do3, do4, do5, do6, do7, s2, s3
- wire segments 292 -> 244
- no-connect marks 1 -> 0

Commit message: Greatly simplify bus selector circuit
Parts:
- removed Q17, Q19, Q56, Q57, Q58, Q59, Q60, Q61, Q62, Q63, Q64, Q65, Q66, Q67, Q68, Q69, Q70, Q71, Q72, Q73, Q74, Q75, Q76, Q77, Q78, Q79, Q80, Q81, Q82, Q83: 2N7000, electrokit:TO-92_Molded_Wide_Inline, symbol Transistor_FET:2N7000
- added Q12, Q8: 2N7000, electrokit:TO-92_Molded_Wide_Inline, symbol Transistor_FET:2N7000
- renumbered Q13 to Q1, Q7 to Q10, Q8 to Q11, Q9 to Q13, Q10 to Q14, Q11 to Q15, Q12 to Q16, Q14 to Q17, Q16 to Q18, Q18 to Q19, Q1 to Q2, Q2 to Q3, Q15 to Q4, Q3 to Q5, Q84 to Q56, Q85 to Q57, Q86 to Q58, Q87 to Q59, Q4 to Q6, Q88 to Q60, Q89 to Q61, Q90 to Q62, Q91 to Q63, Q92 to Q64, Q93 to Q65, Q94 to Q66, Q95 to Q67, Q96 to Q68, Q97 to Q69, Q5 to Q7, Q98 to Q70, Q99 to Q71, Q100 to Q72, Q101 to Q73, Q102 to Q74, Q103 to Q75, Q104 to Q76, Q105 to Q77, Q106 to Q78, Q107 to Q79, Q108 to Q80, Q109 to Q81, Q110 to Q82, Q111 to Q83, Q112 to Q84, Q113 to Q85, Q114 to Q86, Q115 to Q87, Q116 to Q88, Q117 to Q89, Q6 to Q9, Q118 to Q90, Q119 to Q91, Q120 to Q92, Q121 to Q93, Q122 to Q94, Q123 to Q95, Q124 to Q96, Q125 to Q97, Q126 to Q98, Q127 to Q99
Connections:
- net labels added: sa_and, sb_and, sc_and, sd_and
- wire segments 244 -> 252

Commit message: Additional tweaks to bus selector circuit diagram
Parts:
- removed Q11: 2N7000, electrokit:TO-92_Molded_Wide_Inline, symbol Transistor_FET:2N7000
- added JP1: Jumper_2_Open, Connector_PinHeader_2.54mm:PinHeader_1x02_P2.54mm_Vertical, symbol Jumper:Jumper_2_Open
- added JP2: SolderJumper_2_Open, Jumper:SolderJumper-2_P1.3mm_Open_TrianglePad1.0x1.5mm, symbol Jumper:SolderJumper_2_Open
- added Q10: 2N7000, electrokit:TO-92_Molded_Wide_Inline, symbol Transistor_FET:2N7000
- renumbered Q2 to Q1, Q8 to Q11, Q13 to Q12, Q14 to Q13, Q15 to Q14, Q12 to Q15, Q3 to Q2, Q1 to Q3, Q5 to Q4, Q6 to Q5, Q7 to Q6, Q4 to Q7, Q9 to Q8, Q10 to Q9
Connections:
- net labels added: LED_PWR
- wire segments 252 -> 267

Commit message: Add pull-down resistors to bus selector
Parts:
- added R1, R10, R11, R12, R13, R14, R15, R16, R17, R18, R19, R2, R20, R21, R22, R23, R24, R25, R26, R27, R28, R29, R3, R30, R31, R32, R33, R34, R4, R5, R6, R7, R8, R9: R, emlun:R_Axial_DIN0204_L3.6mm_D1.6mm_P5.08mm_Horizontal, symbol Device:R
- renumbered R66 to R100, R67 to R101, R1 to R35, R2 to R36, R3 to R37, R4 to R38, R5 to R39, R6 to R40, R7 to R41, R8 to R42, R9 to R43, R10 to R44, R11 to R45, R12 to R46, R13 to R47, R14 to R48, R15 to R49, R16 to R50, R17 to R51, R18 to R52, R19 to R53, R20 to R54, R21 to R55, R22 to R56, R23 to R57, R24 to R58, R25 to R59, R26 to R60, R27 to R61, R28 to R62, R29 to R63, R30 to R64, R31 to R65, R32 to R66, R33 to R67, R34 to R68, R35 to R69, R36 to R70, R37 to R71, R38 to R72, R39 to R73, R40 to R74, R41 to R75, R42 to R76, R43 to R77, R44 to R78, R45 to R79, R46 to R80, R47 to R81, R48 to R82, R49 to R83, R50 to R84, R51 to R85, R52 to R86, R53 to R87, R54 to R88, R55 to R89, R56 to R90, R57 to R91, R58 to R92, R59 to R93, R60 to R94, R61 to R95, R62 to R96, R63 to R97, R64 to R98, R65 to R99
Connections:
- wire segments 267 -> 293
