File: alu-control-unit/alu-control-unit.sch (KiCad schematic (older format))
At the start: 13 parts, among them J1 Conn_01x08, J2 Conn_01x08, J3 Conn_01x04, J4 Conn_01x01, J5 Conn_01x08, J6 Conn_01x03, J7 PWR-2_pole_power_connector, U1 8-bit-bitwise-logic, U2 4-way-8-bit-bus-selector, U3 8_bit_xor, U4 8_bit_adder, U5 4-way-8-bit-bus-selector, U6 8-input-NOR

Commit message: Replace footprint J2x2-double_2_pole_connector with PWR-double_2_pole_power_connector
Parts:
- J7: footprint emlun:J2x2-double_2_pole_connector -> emlun:PWR-double_2_pole_power_connector
Changed lines of the file:
@@
 F 0 "J7" H 7778 2097 60  0000 L CNN
 F 1 "PWR-2_pole_power_connector" H 7778 1991 60  0000 L CNN
-F 2 "emlun:J2x2-double_2_pole_connector" H 7650 2250 60  0001 C CNN
+F 2 "emlun:PWR-double_2_pole_power_connector" H 7650 2250 60  0001 C CNN
 F 3 "" H 7650 2250 60  0001 C CNN
 	1    7650 2200
