File: alu-control-unit/alu-control-unit.sch (KiCad schematic (older format))
At the start: 13 parts, among them J1 Conn_01x08, J2 Conn_01x08, J3 Conn_01x04, J4 Conn_01x01, J5 Conn_01x08, J6 Conn_01x03, J7 PWR-2_pole_power_connector, U1 8-bit-bitwise-logic, U2 4-way-8-bit-bus-selector, U3 8_bit_xor, U4 8_bit_adder, U5 4-way-8-bit-bus-selector, U6 8-input-NOR

Commit message: Add pull-down resistors to ALU control unit inputs
Parts:
- added R1, R10, R11, R12, R13, R14, R15, R16, R17, R18, R19, R2, R20, R21, R3, R4, R5, R6, R7, R8, R9: R, emlun:R_Axial_DIN0204_L3.6mm_D1.6mm_P5.08mm_Horizontal, symbol Device:R
Connections:
- wire segments 0 -> 21
